File: Hardware/MCP73831_18650Charger/MCP73831_18650Charger.kicad_sch (KiCad schematic)
At the start: 32 parts, among them J1 Conn_01x03, J2 Conn_01x04, Q1 PNP, U1 MCP73831, U2 LT1308, U4 XB7608A

Commit message: Clean up schematics a bit
Parts:
- U1: symbol Angrywasp-IC:MCP73831 -> AngryWasp.General:MCP73831
- U2: symbol Angrywasp-IC:LT1308 -> AngryWasp.General:LT1308
- U4: symbol Angrywasp-IC:XB7608A -> AngryWasp.General:XB7608A
Changed lines of the file:
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@@
 	)
 	(symbol
-		(lib_id "Angrywasp-IC:MCP73831")
+		(lib_id "AngryWasp.General:MCP73831")
 		(at 71.12 39.37 0)
 		(unit 1)
@@
 	)
 	(symbol
-		(lib_id "Angrywasp-IC:LT1308")
+		(lib_id "AngryWasp.General:LT1308")
 		(at 185.42 49.53 0)
 		(unit 1)
@@
 	)
 	(symbol
-		(lib_id "Angrywasp-IC:XB7608A")
+		(lib_id "AngryWasp.General:XB7608A")
 		(at 129.54 81.28 0)
 		(unit 1)
