File: Hardware/MCP73831_LipoCharger/MCP73831_LipoCharger.kicad_sch (KiCad schematic)
At the start: 25 parts, among them J1 Conn_01x09, Q2 P-Channel MOSFET, U2 LT1308, U3 MCP73831

Commit message: Clean up schematics a bit
Parts:
- U2: symbol Angrywasp-IC:LT1308 -> AngryWasp.General:LT1308
- U3: symbol Angrywasp-IC:MCP73831 -> AngryWasp.General:MCP73831
Changed lines of the file:
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@@
 	)
 	(symbol
-		(lib_id "Angrywasp-IC:LT1308")
+		(lib_id "AngryWasp.General:LT1308")
 		(at 240.03 109.22 0)
 		(unit 1)
@@
 	)
 	(symbol
-		(lib_id "Angrywasp-IC:MCP73831")
+		(lib_id "AngryWasp.General:MCP73831")
 		(at 95.25 109.22 0)
 		(unit 1)
