File: Hardware/ESP32_FT232RL_UART/ESP32_FT232RL_UART.kicad_pcb (KiCad board)
At the start: 4 copper layers, 34 x 26 mm, 20 parts, among them J1 Conn_01x06, J2 Conn_01x04, Q1 NPN, Q2 NPN

Commit message: Hardware updates and cleanup
Parts:
- moved R1 2.43 mm to (132.2, 88.0), turned to 90 degrees
- moved R6 0.99 mm to (130.0, 88.0), turned to -90 degrees
Connections:
- Q2 pad 1: IO0 -> DTR
- Q2 pad 3: DTR -> IO0
Routing:
- net IO0: track 6.28 -> 9.51 mm, vias 0 -> 2
- net DTR: track 8.45 -> 11.6 mm
- net EN: track 17.4 -> 18.7 mm
- net Net-(Q2-B): track 5.52 -> 5.86 mm, vias 0 -> 2
- net GND: vias 46 -> 47
Other:
- board text added: "ESP32 FT232RL UART rev. C"
- board text removed: "ESP32 FT232RL UART rev. B"
