File: Hardware/ESP32_FT232RL_UART/ESP32_FT232RL_UART.kicad_sch (KiCad schematic)
At the start: 16 parts, among them J1 Conn_01x06, J2 Conn_01x04, Q1 NPN, Q2 NPN

Commit message: Hardware updates and cleanup
Connections:
- net DTR: now also Q2.1 (E); no longer Q2.3 (C)
- net IO0: now also Q2.3 (C); no longer Q2.1 (E)
Changed lines of the file:
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@@
 		(lib_id "Transistor_BJT:2N3904")
 		(at 240.03 105.41 0)
+		(mirror x)
 		(unit 1)
 		(exclude_from_sim no)
@@
 		(dnp no)
 		(property "Reference" "Q2"
-			(at 245.364 104.902 0)
+			(at 245.364 105.918 0)
 			(effects
 				(font
@@
 		)
 		(property "Value" "NPN"
-			(at 245.872 107.442 0)
+			(at 245.872 103.378 0)
 			(effects
 				(font
@@
 		)
 		(property "Footprint" "Package_TO_SOT_SMD:SOT-23_Handsoldering"
-			(at 245.11 107.315 0)
+			(at 245.11 103.505 0)
 			(effects
 				(font
