File: Hardware/ESP32_Mini/ESP32_Mini.kicad_pcb (KiCad board)
At the start: 4 copper layers, 42 x 42 mm, 20 parts, among them J1 Conn_01x09, J2 Conn_01x09, J3 Conn_01x08, J4 Conn_01x08, SW2 BOOT, SW9 EN, U1 ESP32-S3-WROOM-1

Commit message: Hardware updates and cleanup
Other:
- board text added: "BOOT"
Changed lines of the file:
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@@
 		(layer "Edge.Cuts")
+	)
+	(gr_text "BOOT"
+		(at 136.1 74 90)
+		(layer "F.SilkS")
+		(effects
+			(font
+				(size 1 1)
+				(thickness 0.15)
+			)
+			(justify bottom)
+		)
+	)
+	(gr_text "EN"
+		(at 136.1 86 90)
+		(layer "F.SilkS")
+		(effects
+			(font
+				(size 1 1)
+				(thickness 0.15)
+			)
+			(justify bottom)
+		)
 	)
 	(gr_text "IO40"
