File: Hardware/P8X32A_FT232RL_UART/P8X32A_FT232RL_UART.kicad_sch (KiCad schematic)
At the start: 15 parts, among them J1 Conn_01x05, J2 Conn_01x04, Q2 NPN, U2 74LVC1G126

Commit message: Hardware updates and cleanup
Parts:
- removed U2: 74LVC1G126, symbol 74xGxx:74LVC1G126
Changed lines of the file:
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@@
-	)
-	(symbol
-		(lib_id "74xGxx:74LVC1G126")
-		(at 186.69 123.19 0)
-		(unit 1)
-		(exclude_from_sim no)
-		(in_bom yes)
-		(on_board yes)
-		(dnp no)
-		(fields_autoplaced yes)
-		(property "Reference" "U2"
-			(at 199.39 116.7698 0)
-			(effects
-				(font
-					(size 1.27 1.27)
-				)
-			)
-		)
-		(property "Value" "74LVC1G126"
-			(at 199.39 119.3098 0)
-			(effects
-				(font
-					(size 1.27 1.27)
-				)
-			)
-		)
-		(property "Footprint" ""
-			(at 186.69 123.19 0)
-			(effects
-				(font
-					(size 1.27 1.27)
-				)
-				(hide yes)
-			)
-		)
-		(property "Datasheet" "http://www.ti.com/lit/sg/scyt129e/scyt129e.pdf"
-			(at 186.69 123.19 0)
-			(effects
-				(font
-					(size 1.27 1.27)
-				)
-				(hide yes)
-			)
-		)
-		(property "Description" "Single Buffer Gate Tri-State, Low-Voltage CMOS"
-			(at 186.69 123.19 0)
-			(effects
-				(font
-					(size 1.27 1.27)
-				)
-				(hide yes)
-			)
-		)
-		(pin "3"
-		)
-		(pin "5"
-		)
-		(pin "2"
-		)
-		(pin "1"
-		)
-		(pin "4"
-		)
-		(instances
-			(project ""
-				(path "/6dfbc304-1b3f-4a68-8670-5f15e8ba896c"
-					(reference "U2")
-					(unit 1)
-				)
-			)
-		)
 	)
 	(symbol
