File: Hardware/TPS63000_DcConverter/TPS63000_DcConverter.kicad_sch (KiCad schematic)
At the start: 12 parts, among them J2 Output, J3 Input, U2 TPS63000

Commit message: Hardware updates and cleanup
Parts:
- L1: footprint Inductor_SMD:L_APV_APH0630 -> Inductor_SMD:L_APV_APH0530
Changed lines of the file:
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@@
 			)
 		)
-		(property "Footprint" "Inductor_SMD:L_APV_APH0630"
+		(property "Footprint" "Inductor_SMD:L_APV_APH0530"
 			(at 199.39 82.55 0)
 			(effects
