File: Hardware/ESP32_FT232RL_USBC_UART/ESP32_FT232RL_USBC_UART.kicad_pcb (KiCad board)
At the start: 4 copper layers, 34 x 34 mm, 29 parts, among them J1 USB_C_Receptacle_USB2.0_16P, J2 Conn_01x04, J3 Conn_01x04, Q1 NPN, Q2 NPN, U2 USBLC6-2SC6, U5 74LVC1G126, U6 74LVC1G126

Commit message: Hardware updates. Add Lr04 lora module datasheets
Parts:
- added R10: 100k, Resistor_SMD:R_0805_2012Metric_Pad1.20x1.40mm_HandSolder, F.Cu at (120.7, 80.8)
- added R12: 10k, Resistor_SMD:R_0805_2012Metric_Pad1.20x1.40mm_HandSolder, F.Cu at (128.0, 81.0)
- added R8: 10k, Resistor_SMD:R_0805_2012Metric_Pad1.20x1.40mm_HandSolder, F.Cu at (120.2, 98.5)
- added R9: 10k, Resistor_SMD:R_0805_2012Metric_Pad1.20x1.40mm_HandSolder, F.Cu at (124.0, 81.5)
- moved R6 3.25 mm to (107.8, 98.5)
- moved R5 2.75 mm to (112.2, 98.5)
- moved R7 2.75 mm to (116.2, 98.5)
- moved U2 2.37 mm to (110.0, 81.7)
- moved FB1 2.16 mm to (115.0, 81.0), turned to 180 degrees
- moved C2 1.28 mm to (105.0, 82.0)
Routing:
- net +3.3VA: track 36.0 -> 47.0 mm, vias 3 -> 6
- net RXB: track 5.85 -> 13.8 mm, vias 0 -> 2
- net +5V: track 32.6 -> 28.4 mm
- net TXA: track 10.1 -> 13.1 mm
- net Net-(J1-D+-PadA6): track 6.47 -> 8.84 mm
- net Net-(D2-K): track 24.9 -> 22.7 mm
- net Net-(J1-D--PadA7): track 4.82 -> 6.92 mm
- net D+: track 6.82 -> 4.96 mm
- net D-: track 8.20 -> 7.02 mm
- net Net-(Q1-B): track 12.4 -> 13.6 mm
- net RTS: track 17.2 -> 18.3 mm, vias 2 -> 3
- net IO0: track 20.6 -> 21.5 mm
- net Net-(Q2-B): track 15.0 -> 14.2 mm
- net GND: vias 63 -> 64
- net +3.3V: vias 10 -> 11
Other:
- board text added: "ESP32 USBC-UART rev. B"
- board text removed: "ESP32 USBC-UART rev. A"
