File: Hardware/MCP2221A_USBC_UART/MCP2221A_USBC_UART.kicad_pcb (KiCad board)
At the start: 4 copper layers, 34 x 42 mm, 43 parts, among them J1 USB_C_Receptacle_USB2.0_16P, J2 Output Header, J5 Conn_01x04, Q1 AO3400A, Q2 AO3400A, SW1 SW_PUSH, U1 USBLC6-2SC6, U2 MCP2221AxSL, U3 XC6220B331MR, U4 TCA9517D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

Commit message: Hardware updates. Add Lr04 lora module datasheets
Parts:
- added R18: 10k, Resistor_SMD:R_0805_2012Metric_Pad1.20x1.40mm_HandSolder, F.Cu at (156.0, 134.0)
- added R19: 10k, Resistor_SMD:R_0805_2012Metric_Pad1.20x1.40mm_HandSolder, F.Cu at (166.3, 118.2)
- added R7: 100k, Resistor_SMD:R_0805_2012Metric_Pad1.20x1.40mm_HandSolder, F.Cu at (169.5, 131.0)
- added R8: 10k, Resistor_SMD:R_0805_2012Metric_Pad1.20x1.40mm_HandSolder, F.Cu at (166.3, 121.5)
- moved R4 2.50 mm to (166.1, 114.5), turned to -90 degrees
- moved R16 1.50 mm to (149.0, 135.0)
- moved C5 1.00 mm to (158.0, 136.0)
- moved C6 1.00 mm to (154.0, 136.0)
- moved R1 0.05 mm to (162.5, 122.0)
Routing:
- net TXA: track 5.99 -> 19.3 mm, vias 0 -> 2
- net RXB: track 21.6 -> 23.6 mm, vias 1 -> 2
- net SCLB: track 23.9 -> 25.6 mm
- net TXB: track 22.9 -> 22.5 mm, vias 1 -> 2
- net IOB: track 21.9 -> 21.5 mm, vias 0 -> 1
- net +3.3VA: vias 9 -> 12
- net +3.3V: vias 12 -> 13
Other:
- board text added: "MCP2221A USBC-UART/I2C rev. B"
- board text removed: "MCP2221A USBC-UART/I2C rev. A"
