File: Hardware/P8X32A_AD/P8X32A_AD.kicad_sch (KiCad schematic)
At the start: 20 parts, among them J1 Conn_01x12, J2 Conn_01x12, J3 Conn_01x08, J4 Conn_01x07, SW1 SW_PUSH, U1 Propeller, U2 24LC512, U3 AD7812, Y1 5Mhz

Commit message: Clean up schematics a bit
Parts:
- U1: symbol Angrywasp-IC:Propeller -> AngryWasp.General:Propeller
- U2: symbol Angrywasp-IC:24LC512 -> AngryWasp.General:24LC512
- U3: symbol Angrywasp-IC:AD7812 -> AngryWasp.General:AD7812
Changed lines of the file:
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@@
 	)
 	(symbol
-		(lib_id "Angrywasp-IC:24LC512")
+		(lib_id "AngryWasp.General:24LC512")
 		(at 92.71 60.96 0)
 		(unit 1)
@@
 	)
 	(symbol
-		(lib_id "Angrywasp-IC:AD7812")
+		(lib_id "AngryWasp.General:AD7812")
 		(at 172.72 138.43 0)
 		(unit 1)
@@
 	)
 	(symbol
-		(lib_id "Angrywasp-IC:Propeller")
+		(lib_id "AngryWasp.General:Propeller")
 		(at 53.213 86.36 0)
 		(unit 1)

Commit message: Hardware updates. Add Lr04 lora module datasheets
Parts:
- Y1: footprint Crystal:Crystal_SMD_HC49-SD_HandSoldering -> Crystal:Crystal_SMD_HC49-SD
Changed lines of the file:
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@@
 			)
 		)
-		(property "Footprint" "Crystal:Crystal_SMD_HC49-SD_HandSoldering"
+		(property "Footprint" "Crystal:Crystal_SMD_HC49-SD"
 			(at 72.39 112.395 0)
 			(effects
