File: Hardware/P8X32A_FT232RL_USBC_UART/P8X32A_FT232RL_USBC_UART.kicad_pcb (KiCad board)
At the start: 4 copper layers, 34 x 34 mm, 30 parts, among them J1 USB_C_Receptacle_USB2.0_16P, J2 Conn_01x04, J3 Conn_01x04, Q1 NPN, Q2 NPN, U2 USBLC6-2SC6, U5 74LVC1G126, U6 74LVC1G126

Commit message: Hardware updates. Add Lr04 lora module datasheets
Parts:
- added R10: 10k, Resistor_SMD:R_0805_2012Metric_Pad1.20x1.40mm_HandSolder, F.Cu at (137.9, 77.0)
- added R7: 10k, Resistor_SMD:R_0805_2012Metric_Pad1.20x1.40mm_HandSolder, F.Cu at (134.0, 77.5)
- added R8: 10k, Resistor_SMD:R_0805_2012Metric_Pad1.20x1.40mm_HandSolder, F.Cu at (129.3, 95.2)
- added R9: 100k, Resistor_SMD:R_0805_2012Metric_Pad1.20x1.40mm_HandSolder, F.Cu at (129.2, 77.8)
- moved C5 5.32 mm to (124.3, 94.4), turned to 90 degrees
- moved FB1 2.60 mm to (124.6, 78.0), turned to -90 degrees
- moved U2 1.25 mm to (121.0, 78.2)
- moved R5 1.14 mm to (117.6, 93.8)
- moved R6 0.61 mm to (121.9, 94.4), turned to -90 degrees
Routing:
- net +3.3VA: track 35.1 -> 48.8 mm, vias 3 -> 6
- net TXB: track 5.55 -> 17.1 mm
- net +5V: track 34.2 -> 24.8 mm
- net RXB: track 5.85 -> 13.6 mm, vias 0 -> 2
- net TXA: track 9.27 -> 15.7 mm
- net Net-(D2-K): track 24.9 -> 22.7 mm
- net Net-(D3-K): track 15.0 -> 12.9 mm
- net Net-(Q1-B): track 19.0 -> 17.0 mm
- net Net-(J1-D--PadA7): track 5.02 -> 6.72 mm
- net Net-(J1-D+-PadA6): track 6.69 -> 8.38 mm
- net D+: track 6.74 -> 5.09 mm
- net Net-(Q2-B): track 9.71 -> 8.27 mm
- net Net-(FB1-Pad1): track 8.22 -> 9.33 mm
- net D-: track 8.17 -> 7.38 mm
- net +3.3V: track 4.09 -> 4.23 mm, vias 9 -> 10
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Other:
- board text added: "P8X32A USBC-UART rev. B"
- board text removed: "P8X32A USBC-UART rev. A"
