File: Hardware/P8X32A_FT232RL_USBC_UART/P8X32A_FT232RL_USBC_UART.kicad_sch (KiCad schematic)
At the start: 26 parts, among them J1 USB_C_Receptacle_USB2.0_16P, J2 Conn_01x04, J3 Conn_01x04, Q1 NPN, Q2 NPN, U2 USBLC6-2SC6, U5 74LVC1G126, U6 74LVC1G126

Commit message: Hardware updates. Add Lr04 lora module datasheets
Parts:
- added R10, R7, R8: 10k, Resistor_SMD:R_0805_2012Metric_Pad1.20x1.40mm_HandSolder, symbol Device:R
- added R9: 100k, Resistor_SMD:R_0805_2012Metric_Pad1.20x1.40mm_HandSolder, symbol Device:R
Connections:
- net +3.3V: now also R8.1
- net +3.3VA: now also R10.1, R7.1, R9.2
- net GND: now also R9.1
- net RXB: now also R7.2
- net TXA: now also R8.2
- net TXB: now also R10.2
Other:
- moved on the sheet: J2
