File: Hardware/TB6612FNG_MotorDriver/TB6612FNG_MotorDriver.kicad_sch (KiCad schematic)
At the start: 8 parts, among them J1 01x04, J2 01x04, J3 01x05, J4 01x02, U1 TB6612FNG

Commit message: Hardware updates and cleanup
Parts:
- C1, C2: footprint Capacitor_SMD:C_0805_2012Metric_Pad1.18x1.45mm_HandSolder -> General:0805_HS
- J1, J2: value 01x04 -> Conn_01x04
- J3: value 01x05 -> Conn_01x05
- J4: value 01x02 -> Conn_01x02
Connections:
- net +12V: no longer names the net of C1.1, C3.1, J3.1 (Pin_1), U1.13 (VM2), U1.14 (VM3), U1.24 (VM1)
- net +3.3V: no longer names the net of C2.1, J3.5 (Pin_5), U1.20 (VCC)

Commit message: Hardware updates. Add Lr04 lora module datasheets
Parts:
- C1, C2: footprint General:0805_HS -> Capacitor_SMD:C_0805_2012Metric_Pad1.18x1.45mm_HandSolder
Changed lines of the file:
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@@
 			)
 		)
-		(property "Footprint" "General:0805_HS"
+		(property "Footprint" "Capacitor_SMD:C_0805_2012Metric_Pad1.18x1.45mm_HandSolder"
 			(at 160.02 34.5948 0)
 			(effects
@@
 			)
 		)
-		(property "Footprint" "General:0805_HS"
+		(property "Footprint" "Capacitor_SMD:C_0805_2012Metric_Pad1.18x1.45mm_HandSolder"
 			(at 149.5552 76.2 0)
 			(effects
